Commit message: urdf: joint link need limit
It would not pass `check_urdf` if no limit for joint link

File: practice/robot_descriptionn/urdf/pan_tilt.urdf (robot description, URDF)
Before this commit: robot pan_tilt, 3 links, 2 joints
Joints:
- joint panJoint: limit (none) -> lower=-3.14 upper=3.14 effort=300 velocity=0.1
- joint tiltJoint: limit (none) -> lower=-4.46 upper=-1.5 effort=300 velocity=0.1
